Commit message: add colored model in rviz

File: demo/robot_model/urdf/rosbot.urdf (robot description, URDF)
Before this commit: robot rosbot, 14 links, 13 joints
Links:
- link base_link: geometry collision box size=0.20 0.15 0.04; visual mesh filename=file:/robot_model/meshes/box.stl scale=0.001 0.001 0.001
- link camera_link: geometry collision box size=0.001 0.001 0.001; visual mesh filename=file:/robot_model/meshes/astra.stl scale=0.001 0.001 0.001
- link front_left_wheel: geometry collision mesh filename=file:/robot_model/meshes/wheel.stl scale=0.001 0.001 0.001; visual mesh filename=file:/robot_model/meshes/wheel.stl scale=0.001 0.001 0.001
- link front_right_wheel: geometry collision mesh filename=file:/robot_model/meshes/wheel.stl scale=0.001 0.001 0.001; visual mesh filename=file:/robot_model/meshes/wheel.stl scale=0.001 0.001 0.001
- link laser: geometry collision mesh filename=file:/robot_model/meshes/rplidar.stl scale=0.001 0.001 0.001; visual mesh filename=file:/robot_model/meshes/rplidar.stl scale=0.001 0.001 0.001
- link rear_left_wheel: geometry collision mesh filename=file:/robot_model/meshes/wheel.stl scale=0.001 0.001 0.001; visual mesh filename=file:/robot_model/meshes/wheel.stl scale=0.001 0.001 0.001
- link rear_right_wheel: geometry collision mesh filename=file:/robot_model/meshes/wheel.stl scale=0.001 0.001 0.001; visual mesh filename=file:/robot_model/meshes/wheel.stl scale=0.001 0.001 0.001
- link top: geometry visual mesh filename=file:/robot_model/meshes/upper.stl scale=0.001 0.001 0.001

Commit message: updated robot model

File: demo/robot_model/urdf/rosbot.urdf (robot description, URDF)
Before this commit: robot rosbot, 14 links, 13 joints
Links:
- removed link camera_depth_frame
- removed link camera_rgb_frame
- removed link front_left_wheel
- removed link front_right_wheel
- removed link laser
- removed link range_fl
- removed link range_fr
- removed link range_rl
- removed link range_rr
- removed link rear_left_wheel
- removed link rear_right_wheel
- removed link top
- added link body_link, mass 2.0; collision box size=0.197 0.150 0.080; visual mesh filename=file:/robot_model/meshes/body.stl scale=0.001 0.001 0.001
- added link cover_link, mass 0.000001; visual mesh filename=file:/robot_model/meshes/cover.stl scale=0.001 0.001 0.001
- added link front_left_wheel_link, mass 0.100; collision cylinder length=0.036 radius=0.0425; visual mesh filename=file:/robot_model/meshes/wheel.stl scale=0.001 0.001 0.001
- added link front_right_wheel_link, mass 0.100; collision cylinder length=0.036 radius=0.0425; visual mesh filename=file:/robot_model/meshes/wheel.stl scale=0.001 0.001 0.001
- added link imu_link, mass 0.001
- added link lidar_link, mass 0.190; collision cylinder length=0.0408 radius=0.03625; visual mesh filename=file:/robot_model/meshes/rplidar.stl scale=0.001 0.001 0.001
- added link lidar_link_laser_link
- added link orbbec_astra_depth_link
- added link orbbec_astra_depth_refference_link
- added link orbbec_astra_link, mass 0.105; collision box size=0.165 0.04 0.05; visual mesh filename=file:/robot_model/meshes/astra.stl scale=0.001 0.001 0.001
- added link rear_left_wheel_link, mass 0.100; collision cylinder length=0.036 radius=0.0425; visual mesh filename=file:/robot_model/meshes/wheel.stl scale=0.001 0.001 0.001
- added link rear_right_wheel_link, mass 0.100; collision cylinder length=0.036 radius=0.0425; visual mesh filename=file:/robot_model/meshes/wheel.stl scale=0.001 0.001 0.001
- link base_link: mass 5 -> None; geometry 
- link camera_link: mass 1e-5 -> 0.000001; geometry 
Joints:
- removed joint astra_joint
- removed joint camera_depth_joint
- removed joint camera_optical_joint
- removed joint front_left_wheel_hinge
- removed joint front_right_wheel_hinge
- removed joint range_fl_joint
- removed joint range_fr_joint
- removed joint range_rl_joint
- removed joint range_rr_joint
- removed joint rear_left_wheel_hinge
- removed joint rear_right_wheel_hinge
- removed joint rplidar_joint
- removed joint top_joint
- added joint base_link_to_body_joint: type fixed, parent base_link, child body_link, origin xyz=0.0 0.0 0.0425 rpy=0.0 0.0 0.0
- added joint body_link_to_camera_link_joint: type fixed, parent body_link, child camera_link, origin xyz=-0.0141 0.0 0.125 rpy=0.0 0.0 0.0
- added joint body_link_to_imu_link_joint: type fixed, parent body_link, child imu_link, origin xyz=-0.1369 -0.0419 0.0370 rpy=0.0 0.0 0.0
- added joint body_link_to_lidar_link_joint: type fixed, parent cover_link, child lidar_link, origin xyz=0.02 0.0 0.0 rpy=0.0 0.0 -3.141592653589793
- added joint body_link_to_orbbec_astra_link_joint: type fixed, parent camera_link, child orbbec_astra_link, origin xyz=0.0 0.0 0.0 rpy=0.0 0.0 0.0
- added joint body_to_cover_joint: type fixed, parent body_link, child cover_link, origin xyz=0.0 0.0 0.060 rpy=0.0 0.0 0.0
- added joint front_left_wheel_joint: type continuous, parent body_link, child front_left_wheel_link, origin xyz=0.053 0.096 0.0 rpy=0.0 0.0 0.0, axis 0.0 1.0 0.0, limit effort=1.5 velocity=5.0
- added joint front_right_wheel_joint: type continuous, parent body_link, child front_right_wheel_link, origin xyz=0.053 -0.096 0.0 rpy=0.0 0.0 0.0, axis 0.0 1.0 0.0, limit effort=1.5 velocity=5.0
- added joint lidar_link_laser_link_joint: type fixed, parent lidar_link, child lidar_link_laser_link, origin xyz=0 0 0.0335 rpy=0 0 0
- added joint orbbec_astra_depth_link_joint: type fixed, parent orbbec_astra_link, child orbbec_astra_depth_link, origin xyz=0.01 0 0.035 rpy=0.0 1.5707963267948966 0.0
- added joint orbbec_astra_depth_link_refference_joint: type fixed, parent orbbec_astra_depth_link, child orbbec_astra_depth_refference_link, origin xyz=0.0 0.0 0.0 rpy=1.5707963267948966 -1.5707963267948966 0.0
- added joint rear_left_wheel_joint: type continuous, parent body_link, child rear_left_wheel_link, origin xyz=-0.053 0.096 0.0 rpy=0.0 0.0 0.0, axis 0.0 1.0 0.0, limit effort=1.5 velocity=5.0
- added joint rear_right_wheel_joint: type continuous, parent body_link, child rear_right_wheel_link, origin xyz=-0.053 -0.096 0.0 rpy=0.0 0.0 0.0, axis 0.0 1.0 0.0, limit effort=1.5 velocity=5.0

Commit message: Added ranges to model | updated rosbot_ros

File: demo/robot_model/urdf/rosbot.urdf (robot description, URDF)
Before this commit: robot rosbot, 14 links, 13 joints
Links:
- added link range_left_front
- added link range_left_rear
- added link range_right_front
- added link range_right_rear
Joints:
- added joint range_left_front_joint: type fixed, parent body_link, child range_left_front, origin xyz=0.1 0.05 0.01 rpy=0 0 0.13 , axis 0 1 0
- added joint range_left_rear_joint: type fixed, parent body_link, child range_left_rear, origin xyz=-0.1 0.05 0.01 rpy=0 0 3.01 , axis 0 1 0
- added joint range_right_front_joint: type fixed, parent body_link, child range_right_front, origin xyz=0.1 -0.05 0.01 rpy=0 0 -0.13 , axis 0 1 0
- added joint range_right_rear_joint: type fixed, parent body_link, child range_right_rear, origin xyz=-0.1 -0.05 0.01 rpy=0 0 3.27 , axis 0 1 0

Commit message: added discovery server in an individual container | adjust robot description and nav2 params to ros2

File: demo/robot_model/urdf/rosbot.urdf (robot description, URDF)
Before this commit: robot rosbot, 14 links, 13 joints
Links:
- removed link camera_depth_frame
- removed link camera_rgb_frame
- removed link front_left_wheel
- removed link front_right_wheel
- removed link laser
- removed link range_fl
- removed link range_fr
- removed link range_rl
- removed link range_rr
- removed link rear_left_wheel
- removed link rear_right_wheel
- removed link top
- added link body_link, mass 2.0; collision box size=0.197 0.150 0.080; visual mesh filename=file:/robot_model/meshes/body.stl scale=0.001 0.001 0.001
- added link cover_link, mass 0.000001; visual mesh filename=file:/robot_model/meshes/cover.stl scale=0.001 0.001 0.001
- added link front_left_wheel_link, mass 0.100; collision cylinder length=0.036 radius=0.0425; visual mesh filename=file:/robot_model/meshes/wheel.stl scale=0.001 0.001 0.001
- added link front_right_wheel_link, mass 0.100; collision cylinder length=0.036 radius=0.0425; visual mesh filename=file:/robot_model/meshes/wheel.stl scale=0.001 0.001 0.001
- added link imu_link, mass 0.001
- added link lidar_link, mass 0.190; collision cylinder length=0.0408 radius=0.03625; visual mesh filename=file:/robot_model/meshes/rplidar.stl scale=0.001 0.001 0.001
- added link lidar_link_laser_link
- added link orbbec_astra_depth_link
- added link orbbec_astra_depth_refference_link
- added link orbbec_astra_link, mass 0.105; collision box size=0.165 0.04 0.05; visual mesh filename=file:/robot_model/meshes/astra.stl scale=0.001 0.001 0.001
- added link range_left_front
- added link range_left_rear
- added link range_right_front
- added link range_right_rear
- added link rear_left_wheel_link, mass 0.100; collision cylinder length=0.036 radius=0.0425; visual mesh filename=file:/robot_model/meshes/wheel.stl scale=0.001 0.001 0.001
- added link rear_right_wheel_link, mass 0.100; collision cylinder length=0.036 radius=0.0425; visual mesh filename=file:/robot_model/meshes/wheel.stl scale=0.001 0.001 0.001
- link base_link: mass 5 -> None; geometry 
- link camera_link: mass 1e-5 -> 0.000001; geometry 
Joints:
- removed joint astra_joint
- removed joint camera_depth_joint
- removed joint camera_optical_joint
- removed joint front_left_wheel_hinge
- removed joint front_right_wheel_hinge
- removed joint range_fl_joint
- removed joint range_fr_joint
- removed joint range_rl_joint
- removed joint range_rr_joint
- removed joint rear_left_wheel_hinge
- removed joint rear_right_wheel_hinge
- removed joint rplidar_joint
- removed joint top_joint
- added joint base_link_to_body_joint: type fixed, parent base_link, child body_link, origin xyz=0.0 0.0 0.0425 rpy=0.0 0.0 0.0
- added joint body_link_to_camera_link_joint: type fixed, parent body_link, child camera_link, origin xyz=-0.0141 0.0 0.125 rpy=0.0 0.0 0.0
- added joint body_link_to_imu_link_joint: type fixed, parent body_link, child imu_link, origin xyz=-0.1369 -0.0419 0.0370 rpy=0.0 0.0 0.0
- added joint body_link_to_lidar_link_joint: type fixed, parent cover_link, child lidar_link, origin xyz=0.02 0.0 0.0 rpy=0.0 0.0 -3.141592653589793
- added joint body_link_to_orbbec_astra_link_joint: type fixed, parent camera_link, child orbbec_astra_link, origin xyz=0.0 0.0 0.0 rpy=0.0 0.0 0.0
- added joint body_to_cover_joint: type fixed, parent body_link, child cover_link, origin xyz=0.0 0.0 0.060 rpy=0.0 0.0 0.0
- added joint front_left_wheel_joint: type continuous, parent body_link, child front_left_wheel_link, origin xyz=0.053 0.096 0.0 rpy=0.0 0.0 0.0, axis 0.0 1.0 0.0, limit effort=1.5 velocity=5.0
- added joint front_right_wheel_joint: type continuous, parent body_link, child front_right_wheel_link, origin xyz=0.053 -0.096 0.0 rpy=0.0 0.0 0.0, axis 0.0 1.0 0.0, limit effort=1.5 velocity=5.0
- added joint lidar_link_laser_link_joint: type fixed, parent lidar_link, child lidar_link_laser_link, origin xyz=0 0 0.0335 rpy=0 0 0
- added joint orbbec_astra_depth_link_joint: type fixed, parent orbbec_astra_link, child orbbec_astra_depth_link, origin xyz=0.01 0 0.035 rpy=0.0 1.5707963267948966 0.0
- added joint orbbec_astra_depth_link_refference_joint: type fixed, parent orbbec_astra_depth_link, child orbbec_astra_depth_refference_link, origin xyz=0.0 0.0 0.0 rpy=1.5707963267948966 -1.5707963267948966 0.0
- added joint range_left_front_joint: type fixed, parent body_link, child range_left_front, origin xyz=0.1 0.05 0.01 rpy=0 0 0.13 , axis 0 1 0
- added joint range_left_rear_joint: type fixed, parent body_link, child range_left_rear, origin xyz=-0.1 0.05 0.01 rpy=0 0 3.01 , axis 0 1 0
- added joint range_right_front_joint: type fixed, parent body_link, child range_right_front, origin xyz=0.1 -0.05 0.01 rpy=0 0 -0.13 , axis 0 1 0
- added joint range_right_rear_joint: type fixed, parent body_link, child range_right_rear, origin xyz=-0.1 -0.05 0.01 rpy=0 0 3.27 , axis 0 1 0
- added joint rear_left_wheel_joint: type continuous, parent body_link, child rear_left_wheel_link, origin xyz=-0.053 0.096 0.0 rpy=0.0 0.0 0.0, axis 0.0 1.0 0.0, limit effort=1.5 velocity=5.0
- added joint rear_right_wheel_joint: type continuous, parent body_link, child rear_right_wheel_link, origin xyz=-0.053 -0.096 0.0 rpy=0.0 0.0 0.0, axis 0.0 1.0 0.0, limit effort=1.5 velocity=5.0
